Commit message: Changed name of ROS package

File: urdf/px100.urdf.xacro (robot description, xacro)
@@ -1,32 +1,26 @@
 <?xml version="1.0"?>
 <robot name="px100" xmlns:xacro="http://ros.org/wiki/xacro">
-  <xacro:arg name="use_world_frame" default="false"/>
-  <xacro:arg name="load_gazebo_configs" default="false"/>
   <xacro:property name="pi_offset" value="0.00001"/>
-  <xacro:if value="$(arg load_gazebo_configs)">
-    <xacro:include filename="$(find px100_simulation)/config/px100.gazebo"/>
-  </xacro:if>
+  <xacro:include filename="$(find robomaker_workshop)/config/px100.gazebo"/>
   <material name="interbotix_black">
-    <texture filename="package://px100_simulation/media/materials/textures/interbotix_black.png"/>
+    <texture filename="package://robomaker_workshop/media/materials/textures/interbotix_black.png"/>
   </material>
-  <xacro:if value="$(arg use_world_frame)">
-    <link name="world"/>
-    <joint name="fixed" type="fixed">
-      <parent link="world"/>
-      <child link="px100/base_link"/>
-    </joint>
-  </xacro:if>
+  <link name="world"/>
+  <joint name="fixed" type="fixed">
+    <parent link="world"/>
+    <child link="px100/base_link"/>
+  </joint>
   <link name="px100/base_link">
     <visual>
       <origin rpy="0 0 ${pi/2}" xyz="0 0 0"/>
       <geometry>
-        <mesh filename="package://px100_simulation/meshes/px100_1_base.stl" scale="0.001 0.001 0.001"/>
-      </geometry>
-      <material name="interbotix_black"/>
-    </visual>
-    <collision>
-      <origin rpy="0 0 ${pi/2}" xyz="0 0 0"/>
-      <geometry>
-        <mesh filename="package://px100_simulation/meshes/px100_1_base.stl" scale="0.001 0.001 0.001"/>
+        <mesh filename="package://robomaker_workshop/meshes/px100_1_base.stl" scale="0.001 0.001 0.001"/>
+      </geometry>
+      <material name="interbotix_black"/>
+    </visual>
+    <collision>
+      <origin rpy="0 0 ${pi/2}" xyz="0 0 0"/>
+      <geometry>
+        <mesh filename="package://robomaker_workshop/meshes/px100_1_base.stl" scale="0.001 0.001 0.001"/>
       </geometry>
     </collision>
@@ -58,5 +52,5 @@
       <origin rpy="0 0 ${pi/2}" xyz="0 0 -0.0022"/>
       <geometry>
-        <mesh filename="package://px100_simulation/meshes/px100_2_shoulder.stl" scale="0.001 0.001 0.001"/>
+        <mesh filename="package://robomaker_workshop/meshes/px100_2_shoulder.stl" scale="0.001 0.001 0.001"/>
       </geometry>
       <material name="interbotix_black"/>
@@ -65,5 +59,5 @@
       <origin rpy="0 0 ${pi/2}" xyz="0 0 -0.0022"/>
       <geometry>
-        <mesh filename="package://px100_simulation/meshes/px100_2_shoulder.stl" scale="0.001 0.001 0.001"/>
+        <mesh filename="package://robomaker_workshop/meshes/px100_2_shoulder.stl" scale="0.001 0.001 0.001"/>
       </geometry>
     </collision>
@@ -95,12 +89,12 @@
       <origin rpy="0 0 ${pi/2}" xyz="0 0 0"/>
       <geometry>
-        <mesh filename="package://px100_simulation/meshes/px100_3_upper_arm.stl" scale="0.001 0.001 0.001"/>
-      </geometry>
-      <material name="interbotix_black"/>
-    </visual>
-    <collision>
-      <origin rpy="0 0 ${pi/2}" xyz="0 0 0"/>
-      <geometry>
-        <mesh filename="package://px100_simulation/meshes/px100_3_upper_arm.stl" scale="0.001 0.001 0.001"/>
+        <mesh filename="package://robomaker_workshop/meshes/px100_3_upper_arm.stl" scale="0.001 0.001 0.001"/>
+      </geometry>
+      <material name="interbotix_black"/>
+    </visual>
+    <collision>
+      <origin rpy="0 0 ${pi/2}" xyz="0 0 0"/>
+      <geometry>
+        <mesh filename="package://robomaker_workshop/meshes/px100_3_upper_arm.stl" scale="0.001 0.001 0.001"/>
       </geometry>
     </collision>
@@ -132,12 +126,12 @@
       <origin rpy="0 0 ${pi/2}" xyz="0 0 0"/>
       <geometry>
-        <mesh filename="package://px100_simulation/meshes/px100_4_forearm.stl" scale="0.001 0.001 0.001"/>
-      </geometry>
-      <material name="interbotix_black"/>
-    </visual>
-    <collision>
-      <origin rpy="0 0 ${pi/2}" xyz="0 0 0"/>
-      <geometry>
-        <mesh filename="package://px100_simulation/meshes/px100_4_forearm.stl" scale="0.001 0.001 0.001"/>
+        <mesh filename="package://robomaker_workshop/meshes/px100_4_forearm.stl" scale="0.001 0.001 0.001"/>
+      </geometry>
+      <material name="interbotix_black"/>
+    </visual>
+    <collision>
+      <origin rpy="0 0 ${pi/2}" xyz="0 0 0"/>
+      <geometry>
+        <mesh filename="package://robomaker_workshop/meshes/px100_4_forearm.stl" scale="0.001 0.001 0.001"/>
       </geometry>
     </collision>
@@ -169,12 +163,12 @@
       <origin rpy="0 0 ${pi/2}" xyz="0 0 0"/>
       <geometry>
-        <mesh filename="package://px100_simulation/meshes/px100_5_gripper.stl" scale="0.001 0.001 0.001"/>
-      </geometry>
-      <material name="interbotix_black"/>
-    </visual>
-    <collision>
-      <origin rpy="0 0 ${pi/2}" xyz="0 0 0"/>
-      <geometry>
-        <mesh filename="package://px100_simulation/meshes/px100_5_gripper.stl" scale="0.001 0.001 0.001"/>
+        <mesh filename="package://robomaker_workshop/meshes/px100_5_gripper.stl" scale="0.001 0.001 0.001"/>
+      </geometry>
+      <material name="interbotix_black"/>
+    </visual>
+    <collision>
+      <origin rpy="0 0 ${pi/2}" xyz="0 0 0"/>
+      <geometry>
+        <mesh filename="package://robomaker_workshop/meshes/px100_5_gripper.stl" scale="0.001 0.001 0.001"/>
       </geometry>
     </collision>
@@ -218,5 +212,5 @@
       <origin rpy="0 0 ${pi/2}" xyz="-0.0685 0 0"/>
       <geometry>
-        <mesh filename="package://px100_simulation/meshes/px100_6_gripper_prop.stl" scale="0.001 0.001 0.001"/>
+        <mesh filename="package://robomaker_workshop/meshes/px100_6_gripper_prop.stl" scale="0.001 0.001 0.001"/>
       </geometry>
       <material name="interbotix_black"/>
@@ -225,5 +219,5 @@
       <origin rpy="0 0 ${pi/2}" xyz="-0.0685 0 0"/>
       <geometry>
-        <mesh filename="package://px100_simulation/meshes/px100_6_gripper_prop.stl" scale="0.001 0.001 0.001"/>
+        <mesh filename="package://robomaker_workshop/meshes/px100_6_gripper_prop.stl" scale="0.001 0.001 0.001"/>
       </geometry>
     </collision>
@@ -245,5 +239,5 @@
       <origin rpy="0 0 ${pi/2}" xyz="-0.063 0 0"/>
       <geometry>
-        <mesh filename="package://px100_simulation/meshes/px100_7_gripper_bar.stl" scale="0.001 0.001 0.001"/>
+        <mesh filename="package://robomaker_workshop/meshes/px100_7_gripper_bar.stl" scale="0.001 0.001 0.001"/>
       </geometry>
       <material name="interbotix_black"/>
@@ -252,5 +246,5 @@
       <origin rpy="0 0 ${pi/2}" xyz="-0.063 0 0"/>
       <geometry>
-        <mesh filename="package://px100_simulation/meshes/px100_7_gripper_bar.stl" scale="0.001 0.001 0.001"/>
+        <mesh filename="package://robomaker_workshop/meshes/px100_7_gripper_bar.stl" scale="0.001 0.001 0.001"/>
       </geometry>
     </collision>
@@ -294,5 +288,5 @@
       <origin rpy="${pi} ${pi} 0" xyz="0 0.005 0"/>
       <geometry>
-        <mesh filename="package://px100_simulation/meshes/px100_8_gripper_finger.stl" scale="0.001 0.001 0.001"/>
+        <mesh filename="package://robomaker_workshop/meshes/px100_8_gripper_finger.stl" scale="0.001 0.001 0.001"/>
       </geometry>
       <material name="interbotix_black"/>
@@ -301,5 +295,5 @@
       <origin rpy="${pi} ${pi} 0" xyz="0 0.005 0"/>
       <geometry>
-        <mesh filename="package://px100_simulation/meshes/px100_8_gripper_finger.stl" scale="0.001 0.001 0.001"/>
+        <mesh filename="package://robomaker_workshop/meshes/px100_8_gripper_finger.stl" scale="0.001 0.001 0.001"/>
       </geometry>
     </collision>
@@ -317,7 +311,4 @@
     <child link="px100/right_finger_link"/>
     <dynamics friction="0.1"/>
-    <xacro:unless value="$(arg load_gazebo_configs)">
-      <mimic joint="left_finger" multiplier="-1" offset="0"/>
-    </xacro:unless>
   </joint>
   <transmission name="trans_right_finger">
@@ -334,5 +325,5 @@
       <origin rpy="0 ${pi} 0" xyz="0 -0.005 0"/>
       <geometry>
-        <mesh filename="package://px100_simulation/meshes/px100_8_gripper_finger.stl" scale="0.001 0.001 0.001"/>
+        <mesh filename="package://robomaker_workshop/meshes/px100_8_gripper_finger.stl" scale="0.001 0.001 0.001"/>
       </geometry>
       <material name="interbotix_black"/>
@@ -341,5 +332,5 @@
       <origin rpy="0 ${pi} 0" xyz="0 -0.005 0"/>
       <geometry>
-        <mesh filename="package://px100_simulation/meshes/px100_8_gripper_finger.stl" scale="0.001 0.001 0.001"/>
+        <mesh filename="package://robomaker_workshop/meshes/px100_8_gripper_finger.stl" scale="0.001 0.001 0.001"/>
       </geometry>
     </collision>
